File: zdroj/zdroj.sch (KiCad schematic (older format))
At the start: 10 parts, among them J1 +5V, J2 Molex, J3 Double USB, J4 RD-35A, J5 +12V, U1 IEC_C14_with_switch

Commit message: update README, add pictures
Parts:
- R2: value 1k -> 220
Changed lines of the file:
@@
 P 3900 2550
 F 0 "R2" V 3693 2550 50  0000 C CNN
-F 1 "1k" V 3784 2550 50  0000 C CNN
+F 1 "220" V 3784 2550 50  0000 C CNN
 F 2 "Resistor_THT:R_Axial_DIN0411_L9.9mm_D3.6mm_P20.32mm_Horizontal" V 3830 2550 50  0001 C CNN
 F 3 "~" H 3900 2550 50  0001 C CNN
